File: hardware/Source/nervous-eda.kicad_pcb (KiCad board)
At the start: 2 copper layers, 26 x 40 mm, 55 parts, among them J1 CONN RCP USB3.1 TYPEC 24P SMD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, J2 MOLEX 53048-0310, J4 CONN HEADER R/A 4POS 2.54MM, U1 SWITCH TACTILE SPST-NO 0.02A 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, U10 IC MCU 32BIT 32KB FLASH 28SSOP, U2 TVS Diode WE-TVS-Standard, VR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, U3 IC INTFACE SPECIALIZED TSOT23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, U4 IC BATT CHG LI-ION 1CELL 16QFN, U5 IC REG LINEAR 3.3V 200MA SOT2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, U6 IC BATT FUEL GAUGE LICOO2 12S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

Commit message: fix : readjustment of decoupling capacity positioning
Parts:
- moved C12 15.9 mm to (48.2, 44.0)
- moved C9 11.5 mm to (43.6, 38.0), turned to 0 degrees
- moved C8 11.3 mm to (41.0, 38.0), turned to 180 degrees
- moved C14 9.43 mm to (45.9, 49.3), turned to 180 degrees
- moved C13 4.45 mm to (50.6, 44.0), turned to 0 degrees
- moved C15 2.09 mm to (36.6, 30.6)
- moved R16 2.09 mm to (36.6, 32.7)
- moved C7 1.83 mm to (37.6, 28.0), turned to -90 degrees
Routing:
- net VCC: track 81.6 -> 98.6 mm
- net GND: track 60.4 -> 55.2 mm, vias 19 -> 20
- net ZIN: track 13.1 -> 17.2 mm
- net VDD: track 10.6 -> 13.8 mm
- net Net-(U1-NO_1): track 16.1 -> 13.8 mm
- net Net-(U4-~{CHG}): track 31.0 -> 29.3 mm
- net IOUT: track 16.2 -> 14.7 mm
- net SWCLK_PSOC: track 20.4 -> 19.2 mm
- net VBUS: track 14.9 -> 16.1 mm
- net VSYS: track 56.7 -> 57.9 mm
- net VREF: track 14.7 -> 13.7 mm
- net SWDIO_PSOC: track 24.3 -> 23.5 mm
- net Net-(J1-CC1): track 8.56 -> 7.92 mm
- net Net-(J1-CC2): track 11.3 -> 10.7 mm

Commit message: feat: bump to KiCad 9.0.0
Other:
- board text added: "NERVOUS EDA Sensor v1.0.1 RENFORCE-ANR-22-CE31-0023-03 (c) 2024 INSA Lyon, CNRS"
- board text removed: "NERVOUS EDA Sensor v1.0 RENFORCE-ANR-22-CE31-0023-03 (c) 2024 INSA Lyon, CNRS"
