File: hardware/Source/nervous-eda.kicad_pcb (KiCad board)
At the start: 2 copper layers, 26 x 40 mm, 55 parts, among them J1 CONN RCP USB3.1 TYPEC 24P SMD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, J2 MOLEX 53048-0310, J4 CONN HEADER R/A 4POS 2.54MM, U1 SWITCH TACTILE SPST-NO 0.02A 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, U10 IC MCU 32BIT 32KB FLASH 28SSOP, U2 TVS Diode WE-TVS-Standard, VR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, U3 IC INTFACE SPECIALIZED TSOT23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, U4 IC BATT CHG LI-ION 1CELL 16QFN, U5 IC REG LINEAR 3.3V 200MA SOT2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, U6 IC BATT FUEL GAUGE LICOO2 12S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

Commit message: fix: [hw] cosmetics, export files and version update
Parts:
- J4: footprint nervous-eda:CONN_ELECTRODE -> Connector_PinHeader_2.54mm:PinHeader_1x02_P2.54mm_Horizontal
- moved J4 2.54 mm to (33.0, 32.5), turned to 180 degrees
- renumbered U8 to J3, U9 to J5
Connections:
- J4 pad 1: ZOUT -> ZIN
- J4 pad 2: ZIN -> ZOUT
Other:
- board text added: "NERVOUS EDA Sensor v1.1.2 RENFORCE-ANR-22-CE31-0023-03 (c) 2024 INSA Lyon, CNRS"
- board text removed: "NERVOUS EDA Sensor v1.0.1 RENFORCE-ANR-22-CE31-0023-03 (c) 2024 INSA Lyon, CNRS"
