File: hardware/Source/nervous-eda.kicad_sch (KiCad schematic)
At the start: 56 parts, among them J1 CONN RCP USB3.1 TYPEC 24P SMD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, J2 MOLEX 53048-0310, J4 CONN HEADER R/A 4POS 2.54MM, U1 SWITCH TACTILE SPST-NO 0.02A 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, U10 IC MCU 32BIT 32KB FLASH 28SSOP, U11 LIGHTPIPE PNL MT CONVEX 0.250", U12 LIGHTPIPE PNL MT CONVEX 0.250", U2 TVS Diode WE-TVS-Standard, VR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, U3 IC INTFACE SPECIALIZED TSOT23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, U4 IC BATT CHG LI-ION 1CELL 16QFN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

Commit message: fix : readjustment of decoupling capacity positioning
Parts:
- BT1: value BATT LI-PO 3.7V 165MAH -> BATT LI-PO 3.7V 165MAH

Commit message: feat: bump to KiCad 9.0.0
Parts:
- C1, C10, C11, C12, C13, C14, C15, C16, C2, C3, C4, C5, C6, C7, C8, C9: symbol nervous-ecg:C -> nervous-eda:C
- D1: symbol nervous-ecg:D_Schottky -> nervous-eda:D_Schottky
- D4, D5: symbol nervous-ecg:APHF1608LSEEQBDZGKC -> nervous-eda:APHF1608LSEEQBDZGKC
- F1: symbol nervous-ecg:Fuse -> nervous-eda:Fuse
- J1: symbol nervous-ecg:CONN_USB_3.1_TYPE_C_-_105450-0101 -> nervous-eda:CONN_USB_3.1_TYPE_C_-_105450-0101
- J2: symbol nervous-ecg:Conn_01x03_Pin -> nervous-eda:Conn_01x03_Pin
- R1, R10, R11, R12, R13, R14, R15, R16, R17, R19, R3, R5, R6, R7, R8, R9: symbol nervous-ecg:R -> nervous-eda:R
- U1: symbol nervous-ecg:EVP-AA502W -> nervous-eda:EVP-AA502W
- U2: symbol nervous-ecg:TVS_DIODE_5VWM_SOT23-3L_1 -> nervous-eda:TVS_DIODE_5VWM_SOT23-3L_1
- U3: symbol nervous-ecg:MAX16054AZT+T -> nervous-eda:MAX16054AZT+T
- U4: symbol nervous-ecg:BQ24074RGTT -> nervous-eda:BQ24074RGTT
- U5: symbol nervous-ecg:TPS7A0533PDBVR -> nervous-eda:TPS7A0533PDBVR
- U6: symbol nervous-ecg:BQ27441DRZT-G1A -> nervous-eda:BQ27441DRZT-G1A
- U7: symbol nervous-ecg:ISP1807-LR -> nervous-eda:ISP1807-LR
- U8, U9: symbol nervous-ecg:TC2030-MCP-NL -> nervous-eda:TC2030-MCP-NL

Commit message: fix: [hw] cosmetics, export files and version update
Parts:
- C15, C16: now not fitted; now left out of the parts list
- J4: footprint nervous-eda:CONN_ELECTRODE -> Connector_PinHeader_2.54mm:PinHeader_1x02_P2.54mm_Horizontal
- R16: now not fitted
- renumbered U8 to J3, U9 to J5
Connections:
- net ZIN: now also J4.1 (Pin_1); no longer J4.2 (Pin_2)
- net ZOUT: now also J4.2 (Pin_2); no longer J4.1 (Pin_1)
Changed lines of the file:
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@@
 		(title "NERVOUS - EDA Sensor")
 		(date "2025-03-20")
-		(rev "1")
+		(rev "1.1.2")
 		(comment 1 "Copyright (c) 2024 INSA Lyon, CNRS, INL UMR5270")
 		(comment 2 "License : MIT License")
@@
 	(text_box "BQ24074 Configuration :\n\nRset = 5.93k  (Iset (155mA max) = 890 / Rset)\nRlim = 3.05k  (Ilim (500mA max) = 1525 / Rlim)\nDo not mount R5 if battery pack has 10k thermistor"
 		(exclude_from_sim no)
-		(at 100.33 38.1 0)
-		(size 44.45 12.7)
+		(at 88.9 30.48 0)
+		(size 55.88 12.7)
 		(margins 0.9525 0.9525 0.9525 0.9525)
 		(stroke
@@
 	(wire
 		(pts
+			(xy 209.55 227.33) (xy 214.63 227.33)
+		)
+		(stroke
+			(width 0)
+			(type default)
+		)
+	)
+	(wire
+		(pts
 			(xy 394.97 106.68) (xy 374.65 106.68)
 		)
@@
 	(wire
 		(pts
-			(xy 209.55 227.33) (xy 214.63 227.33)
-		)
-		(stroke
-			(width 0)
-			(type default)
-		)
-	)
-	(wire
-		(pts
 			(xy 123.19 71.12) (xy 123.19 59.69)
 		)
@@
 	(wire
 		(pts
+			(xy 209.55 224.79) (xy 214.63 224.79)
+		)
+		(stroke
+			(width 0)
+			(type default)
+		)
+	)
+	(wire
+		(pts
 			(xy 266.7 175.26) (xy 266.7 170.18)
 		)
@@
 	(wire
 		(pts
-			(xy 209.55 224.79) (xy 214.63 224.79)
-		)
-		(stroke
-			(width 0)
-			(type default)
-		)
-	)
-	(wire
-		(pts
 			(xy 119.38 143.51) (xy 119.38 138.43)
 		)
@@
 				)
 			)
-			(project "nervous-eda"
-				(path "/f891394e-87c7-4671-ba51-f289fceaf1a5"
-					(reference "C5")
-					(unit 1)
-				)
-			)
 		)
 	)
@@
 				)
 			)
-			(project "nervous-eda"
-				(path "/f891394e-87c7-4671-ba51-f289fceaf1a5"
-					(reference "H1")
-					(unit 1)
-				)
-			)
 		)
 	)
@@
 		(dnp no)
 		(fields_autoplaced yes)
-		(property "Reference" "U9"
-			(at 367.03 205.74 0)
+		(property "Reference" "J5"
+			(at 367.03 203.2 0)
 			(effects
 				(font
@@
 		)
 		(property "Value" "~"
-			(at 359.41 212.09 0)
+			(at 367.03 205.74 0)
 			(effects
 				(font
@@
 			(project "nervous-eda"
 				(path "/13e5af92-cf6a-4e6a-aa06-08418eba810e"
-					(reference "U9")
+					(reference "J5")
 					(unit 1)
 				)
@@
 				)
 			)
-			(project "nervous-eda"
-				(path "/f891394e-87c7-4671-ba51-f289fceaf1a5"
-					(reference "H2")
-					(unit 1)
-				)
-			)
 		)
 	)
@@
 	)
 	(symbol
+		(lib_name "TC2030-MCP-NL_1")
 		(lib_id "nervous-eda:TC2030-MCP-NL")
 		(at 367.03 184.15 0)
@@
 		(dnp no)
 		(fields_autoplaced yes)
-		(property "Reference" "U8"
-			(at 367.03 177.8 0)
+		(property "Reference" "J3"
+			(at 367.03 175.26 0)
 			(effects
 				(font
@@
 		)
 		(property "Value" "~"
-			(at 359.41 184.15 0)
+			(at 367.03 177.8 0)
 			(effects
 				(font
@@
 			(project "nervous-eda"
 				(path "/13e5af92-cf6a-4e6a-aa06-08418eba810e"
-					(reference "U8")
+					(reference "J3")
 					(unit 1)
 				)
@@
 		(in_bom no)
 		(on_board yes)
-		(dnp no)
+		(dnp yes)
 		(property "Reference" "R16"
 			(at 240.03 223.52 0)
@@
 		(unit 1)
 		(exclude_from_sim no)
-		(in_bom yes)
+		(in_bom no)
 		(on_board yes)
-		(dnp no)
+		(dnp yes)
 		(property "Reference" "C16"
 			(at 298.45 226.06 90)
@@
 		(unit 1)
 		(exclude_from_sim no)
-		(in_bom yes)
+		(in_bom no)
 		(on_board yes)
-		(dnp no)
+		(dnp yes)
 		(property "Reference" "C15"
 			(at 227.33 223.52 0)
@@
 	(symbol
 		(lib_id "nervous-eda:CONN_ELECTRODES")
-		(at 204.47 227.33 0)
+		(at 204.47 224.79 0)
+		(mirror x)
 		(unit 1)
 		(exclude_from_sim no)
@@
 		)
 		(property "Value" "CONN HEADER R/A 4POS 2.54MM"
-			(at 191.77 231.14 0)
+			(at 191.77 220.98 0)
 			(effects
 				(font
@@
 			)
 		)
-		(property "Footprint" "nervous-eda:CONN_ELECTRODE"
-			(at 204.47 227.33 0)
+		(property "Footprint" "Connector_PinHeader_2.54mm:PinHeader_1x02_P2.54mm_Horizontal"
+			(at 204.47 224.79 0)
 			(effects
 				(font
@@
 		)
 		(property "Datasheet" "~"
-			(at 204.47 227.33 0)
+			(at 204.47 224.79 0)
 			(effects
 				(font
@@
 		)
 		(property "Description" ""
-			(at 204.47 227.33 0)
+			(at 204.47 224.79 0)
 			(effects
 				(font
@@
 		)
 		(property "Manufacturer" "AMPHENOL COMMUNICATIONS SOLUTIONS"
-			(at 204.47 227.33 0)
+			(at 204.47 224.79 0)
 			(effects
 				(font
@@
 		)
 		(property "Manufacturer Part Number" "77315-118-04LF"
-			(at 204.47 227.33 0)
+			(at 204.47 224.79 0)
 			(effects
 				(font
@@
 		)
 		(property "Supplier" "FARNELL"
-			(at 204.47 227.33 0)
+			(at 204.47 224.79 0)
 			(effects
 				(font
@@
 		)
 		(property "Supplier Part Number" "3728851"
-			(at 204.47 227.33 0)
+			(at 204.47 224.79 0)
 			(effects
 				(font
@@
 		)
 		(property "Note" "CONN ELECTRODES"
-			(at 193.04 229.87 0)
+			(at 193.04 222.25 0)
 			(effects
 				(font
